File: KiCad/Projet/Projet.kicad_pcb (KiCad board)
At the start: 2 copper layers, 2 parts, among them U1 WeMos_D1_mini

Commit message: Rain counter OK
Parts:
- added FlowControler1: Cable_01x03_Female, Connector_Wire:SolderWire-0.25sqmm_1x03_P4.2mm_D0.65mm_OD1.7mm, F.Cu at (105.0, 119.4)
- added FlowControlerSignalResistor1: R200ohm, Resistor_THT:R_Axial_DIN0204_L3.6mm_D1.6mm_P7.62mm_Horizontal, F.Cu at (121.9, 99.1)
- added RainControler1: Cable_01x02_Female, Connector_Wire:SolderWire-0.25sqmm_1x02_P4.5mm_D0.65mm_OD2mm, F.Cu at (105.4, 76.2)
- added RainControlerSignalResistor1: R200ohm, Resistor_THT:R_Axial_DIN0204_L3.6mm_D1.6mm_P7.62mm_Horizontal, F.Cu at (121.9, 85.1)
- moved TH_NTC1 29.6 mm to (105.4, 87.6)
Connections:
- net Net-(TH_NTC1-Pad1) renamed /ThermistorSignal
- net Net-(TH_NTC1-Pad3) renamed GND
- U1 pad 5: Net-(U1-Pad5) -> /RainSignal
